Commit message: repo add

File: description/urdf/chitrak_full.urdf (robot description, URDF)
Before this commit: robot chitrak_description, 14 links, 13 joints
Links:
- link bl_calf_link: geometry collision mesh filename=../meshes/bl_calf_link.STL; visual mesh filename=../meshes/bl_calf_link.STL
- link bl_hip_link: geometry collision mesh filename=../meshes/bl_hip_link.STL; visual mesh filename=../meshes/bl_hip_link.STL
- link bl_thigh_link: geometry collision mesh filename=../meshes/bl_thigh_link.STL; visual mesh filename=../meshes/bl_thigh_link.STL
- link br_calf_link: geometry collision mesh filename=../meshes/br_calf_link.STL; visual mesh filename=../meshes/br_calf_link.STL
- link br_hip_link: geometry collision mesh filename=../meshes/br_hip_link.STL; visual mesh filename=../meshes/br_hip_link.STL
- link br_thigh_link: geometry collision mesh filename=../meshes/br_thigh_link.STL; visual mesh filename=../meshes/br_thigh_link.STL
- link fl_calf_link: geometry collision mesh filename=../meshes/fl_calf_link.STL; visual mesh filename=../meshes/fl_calf_link.STL
- link fl_hip_link: geometry collision mesh filename=../meshes/fl_hip_link.STL; visual mesh filename=../meshes/fl_hip_link.STL
- link fl_thigh_link: geometry collision mesh filename=../meshes/fl_thigh_link.STL; visual mesh filename=../meshes/fl_thigh_link.STL
- link fr_calf_link: geometry collision mesh filename=../meshes/fr_calf_link.STL; visual mesh filename=../meshes/fr_calf_link.STL
- link fr_hip_link: geometry collision mesh filename=../meshes/fr_hip_link.STL; visual mesh filename=../meshes/fr_hip_link.STL
- link fr_thigh_link: geometry collision mesh filename=../meshes/fr_thigh_link.STL; visual mesh filename=../meshes/fr_thigh_link.STL
- link torso_link: geometry collision mesh filename=../meshes/torso_link.STL; visual mesh filename=../meshes/torso_link.STL
